Commit message: Simplify iCubGazeboV2_5_vision_manip
Remove control of legs and all sensors

File: iCub/robots/iCubGazeboV2_5_vision_manip/model.urdf (robot description, URDF)
Before this commit: robot iCub, 189 links, 188 joints
Links:
- removed link base_link
Joints:
- removed joint base_fixed_joint

Commit message: Add visual and collision for right/left hand palm and cover
Inertias to be revised

Top cover missing for the right hand

File: iCub/robots/iCubGazeboV2_5_vision_manip/model.urdf (robot description, URDF)
Before this commit: robot iCub, 188 links, 187 joints
Links:
- link l_hand: geometry collision mesh filename=package://iCub/meshes/hand/full_LeftHandPalm.obj scale=1.0 1.0 1.0; collision mesh filename=package://iCub/meshes/hand/full_LeftTopCover.obj scale=1.0 1.0 1.0
- link r_hand: geometry collision mesh filename=package://iCub/meshes/hand/full_RightHandPalm.obj scale=1.0 1.0 1.0; visual mesh filename=package://iCub/meshes/hand/full_RightHandPalm.obj scale=1.0 1.0 1.0

Commit message: Implement left hand in iCubGazeboV2_5_vision_manip

File: iCub/robots/iCubGazeboV2_5_vision_manip/model.urdf (robot description, URDF)
Before this commit: robot iCub, 188 links, 187 joints
Links:
- added link l_hand_index_0, mass 0.01; collision mesh filename=package://iCub/meshes/hand/full_LeftIndex0.obj scale=1.0 1.0 1.0; visual mesh filename=package://iCub/meshes/hand/full_LeftIndex0.obj scale=1.0 1.0 1.0
- added link l_hand_index_1, mass 0.01; collision mesh filename=package://iCub/meshes/hand/full_LeftIndex1.obj scale=1.0 1.0 1.0; visual mesh filename=package://iCub/meshes/hand/full_LeftIndex1.obj scale=1.0 1.0 1.0
- added link l_hand_index_2, mass 0.01; collision mesh filename=package://iCub/meshes/hand/full_LeftIndex2.obj scale=1.0 1.0 1.0; visual mesh filename=package://iCub/meshes/hand/full_LeftIndex2.obj scale=1.0 1.0 1.0
- added link l_hand_index_3, mass 0.01; collision mesh filename=package://iCub/meshes/hand/full_LeftIndex3.obj scale=1.0 1.0 1.0; visual mesh filename=package://iCub/meshes/hand/full_LeftIndex3.obj scale=1.0 1.0 1.0
- added link l_hand_little_0, mass 0.01; collision mesh filename=package://iCub/meshes/hand/full_LeftLittle0.obj scale=1.0 1.0 1.0; visual mesh filename=package://iCub/meshes/hand/full_LeftLittle0.obj scale=1.0 1.0 1.0
- added link l_hand_little_1, mass 0.01; collision mesh filename=package://iCub/meshes/hand/full_LeftLittle1.obj scale=1.0 1.0 1.0; visual mesh filename=package://iCub/meshes/hand/full_LeftLittle1.obj scale=1.0 1.0 1.0
- added link l_hand_little_2, mass 0.01; collision mesh filename=package://iCub/meshes/hand/full_LeftLittle2.obj scale=1.0 1.0 1.0; visual mesh filename=package://iCub/meshes/hand/full_LeftLittle2.obj scale=1.0 1.0 1.0
- added link l_hand_little_3, mass 0.01; collision mesh filename=package://iCub/meshes/hand/full_LeftLittle3.obj scale=1.0 1.0 1.0; visual mesh filename=package://iCub/meshes/hand/full_LeftLittle3.obj scale=1.0 1.0 1.0
- added link l_hand_middle_0, mass 0.01; collision mesh filename=package://iCub/meshes/hand/full_LeftMiddle0.obj scale=1.0 1.0 1.0; visual mesh filename=package://iCub/meshes/hand/full_LeftMiddle0.obj scale=1.0 1.0 1.0
- added link l_hand_middle_1, mass 0.01; collision mesh filename=package://iCub/meshes/hand/full_LeftMiddle1.obj scale=1.0 1.0 1.0; visual mesh filename=package://iCub/meshes/hand/full_LeftMiddle1.obj scale=1.0 1.0 1.0
- added link l_hand_middle_2, mass 0.01; collision mesh filename=package://iCub/meshes/hand/full_LeftMiddle2.obj scale=1.0 1.0 1.0; visual mesh filename=package://iCub/meshes/hand/full_LeftMiddle2.obj scale=1.0 1.0 1.0
- added link l_hand_middle_3, mass 0.01; collision mesh filename=package://iCub/meshes/hand/full_LeftMiddle3.obj scale=1.0 1.0 1.0; visual mesh filename=package://iCub/meshes/hand/full_LeftMiddle3.obj scale=1.0 1.0 1.0
- added link l_hand_ring_0, mass 0.01; collision mesh filename=package://iCub/meshes/hand/full_LeftRing0.obj scale=1.0 1.0 1.0; visual mesh filename=package://iCub/meshes/hand/full_LeftRing0.obj scale=1.0 1.0 1.0
- added link l_hand_ring_1, mass 0.01; collision mesh filename=package://iCub/meshes/hand/full_LeftRing1.obj scale=1.0 1.0 1.0; visual mesh filename=package://iCub/meshes/hand/full_LeftRing1.obj scale=1.0 1.0 1.0
- added link l_hand_ring_2, mass 0.01; collision mesh filename=package://iCub/meshes/hand/full_LeftRing2.obj scale=1.0 1.0 1.0; visual mesh filename=package://iCub/meshes/hand/full_LeftRing2.obj scale=1.0 1.0 1.0
- added link l_hand_ring_3, mass 0.01; collision mesh filename=package://iCub/meshes/hand/full_LeftRing3.obj scale=1.0 1.0 1.0; visual mesh filename=package://iCub/meshes/hand/full_LeftRing3.obj scale=1.0 1.0 1.0
- added link l_hand_thumb_0, mass 0.01; collision mesh filename=package://iCub/meshes/hand/full_LeftThumb0.obj scale=1.0 1.0 1.0; visual mesh filename=package://iCub/meshes/hand/full_LeftThumb0.obj scale=1.0 1.0 1.0
- added link l_hand_thumb_1, mass 0.01; collision mesh filename=package://iCub/meshes/hand/full_LeftThumb1.obj scale=1.0 1.0 1.0; visual mesh filename=package://iCub/meshes/hand/full_LeftThumb1.obj scale=1.0 1.0 1.0
- added link l_hand_thumb_2, mass 0.01; collision mesh filename=package://iCub/meshes/hand/full_LeftThumb2.obj scale=1.0 1.0 1.0; visual mesh filename=package://iCub/meshes/hand/full_LeftThumb2.obj scale=1.0 1.0 1.0
- added link l_hand_thumb_3, mass 0.01; collision mesh filename=package://iCub/meshes/hand/full_LeftThumb3.obj scale=1.0 1.0 1.0; visual mesh filename=package://iCub/meshes/hand/full_LeftThumb3.obj scale=1.0 1.0 1.0
- link l_hand_dh_frame: mass None -> 0.001
Joints:
- added joint l_hand_index_0_joint: type revolute, parent l_hand_dh_frame, child l_hand_index_0, origin xyz=0.00175 -0.02622 0.0107 rpy=0.0870442565935125 3.13536120039556 3.07030553260709, axis 0.0 0.0 1.0, limit lower=0.0 upper=0.3490658503988659 effort=50000 velocity=50000
- added joint l_hand_index_1_joint: type revolute, parent l_hand_index_0, child l_hand_index_1, origin xyz=0.0148 -0.00175 1.07156594925393e-19 rpy=1.5707963267949 0.0 0.0, axis 0.0 0.0 1.0, limit lower=0.0 upper=1.5707963267948966 effort=50000 velocity=50000
- added joint l_hand_index_2_joint: type revolute, parent l_hand_index_1, child l_hand_index_2, origin xyz=0.0259 0.0 0.0 rpy=0.0 0.0 0.0, axis 0.0 0.0 1.0, limit lower=0.0 upper=1.5707963267948966 effort=50000 velocity=50000
- added joint l_hand_index_3_joint: type revolute, parent l_hand_index_2, child l_hand_index_3, origin xyz=0.022 0.0 0.0 rpy=0.0 0.0 0.0, axis 0.0 0.0 1.0, limit lower=0.0 upper=1.5707963267948966 effort=50000 velocity=50000
- added joint l_hand_little_0_joint: type revolute, parent l_hand_dh_frame, child l_hand_little_0, origin xyz=-0.000390000000000001 0.02454 0.01 rpy=-3.13229601984498  0.0867711076126969 0.106868680136788, axis 0.0 0.0 1.0, limit lower=0.0 upper=0.3490658503988659 effort=50000 velocity=50000
- added joint l_hand_little_1_joint: type revolute, parent l_hand_little_0, child l_hand_little_1, origin xyz=0.0148 0.00175 -1.07156594925393e-19 rpy=1.5707963267949 0.0 0.0, axis 0.0 0.0 1.0, limit lower=0.0 upper=1.5707963267948966 effort=50000 velocity=50000
- added joint l_hand_little_2_joint: type revolute, parent l_hand_little_1, child l_hand_little_2, origin xyz=0.0219 0.0 0.0 rpy=0.0 0.0 0.0, axis 0.0 0.0 1.0, limit lower=0.0 upper=1.5707963267948966 effort=50000 velocity=50000
- added joint l_hand_little_3_joint: type revolute, parent l_hand_little_2, child l_hand_little_3, origin xyz=0.019 0.0 0.0 rpy=0.0 0.0 0.0, axis 0.0 0.0 1.0, limit lower=0.0 upper=1.5707963267948966 effort=50000 velocity=50000
- added joint l_hand_middle_0_joint: type revolute, parent l_hand_dh_frame, child l_hand_middle_0, origin xyz=0.0025 -0.00977 0.0116 rpy=3.14159265358979 0.0 0.0, axis 0.0 0.0 1.0, limit lower=0.0 upper=0.3490658503988659 effort=50000 velocity=50000
- added joint l_hand_middle_1_joint: type revolute, parent l_hand_middle_0, child l_hand_middle_1, origin xyz=0.0153 -0.0022 1.34711147906209e-19 rpy=1.5707963267949 0.0 0.0, axis 0.0 0.0 1.0, limit lower=0.0 upper=1.5707963267948966 effort=50000 velocity=50000
- added joint l_hand_middle_2_joint: type revolute, parent l_hand_middle_1, child l_hand_middle_2, origin xyz=0.0258 0.0 0.0 rpy=0.0 0.0 0.0, axis 0.0 0.0 1.0, limit lower=0.0 upper=1.5707963267948966 effort=50000 velocity=50000
- added joint l_hand_middle_3_joint: type revolute, parent l_hand_middle_2, child l_hand_middle_3, origin xyz=0.024 0.0 0.0 rpy=0.0 0.0 0.0, axis 0.0 0.0 1.0, limit lower=0.0 upper=1.5707963267948966 effort=50000 velocity=50000
- added joint l_hand_ring_0_joint: type revolute, parent l_hand_dh_frame, child l_hand_ring_0, origin xyz=0.00163000000000001 0.00565 0.011 rpy=-3.13229601984498 0.0867711076126969  0.106868680136788, axis 0.0 0.0 1.0, limit lower=0.0 upper=0.3490658503988659 effort=50000 velocity=50000
- added joint l_hand_ring_1_joint: type revolute, parent l_hand_ring_0, child l_hand_ring_1, origin xyz= 0.0148 -0.00175 1.07156594925393e-19 rpy=1.5707963267949 0.0 0.0, axis 0.0 0.0 1.0, limit lower=0.0 upper=1.5707963267948966 effort=50000 velocity=50000
- added joint l_hand_ring_2_joint: type revolute, parent l_hand_ring_1, child l_hand_ring_2, origin xyz=0.0259 0.0 0.0 rpy=0.0 0.0 0.0, axis 0.0 0.0 1.0, limit lower=0.0 upper=1.5707963267948966 effort=50000 velocity=50000
- added joint l_hand_ring_3_joint: type revolute, parent l_hand_ring_2, child l_hand_ring_3, origin xyz=0.022 0.0 0.0 rpy=0.0 0.0 0.0, axis 0.0 0.0 1.0, limit lower=0.0 upper=1.5707963267948966 effort=50000 velocity=50000
- added joint l_hand_thumb_0_joint: type revolute, parent l_hand_dh_frame, child l_hand_thumb_0, origin xyz=-0.0235 -0.012 0.0015 rpy=1.6435245522555 -3.10126979642577 2.07617279145347, axis 0.0 0.0 1.0, limit lower=0.0 upper=1.5707963267948966 effort=50000 velocity=50000
- added joint l_hand_thumb_1_joint: type revolute, parent l_hand_thumb_0, child l_hand_thumb_1, origin xyz=0.0211 0.0049 -3.00038465791102e-19 rpy=1.5707963267949 0.0 0.0, axis 0.0 0.0 1.0, limit lower=0.0 upper=1.5707963267948966 effort=50000 velocity=50000
- added joint l_hand_thumb_2_joint: type revolute, parent l_hand_thumb_1, child l_hand_thumb_2, origin xyz=0.026 0.0 0.0 rpy=0.0 0.0 0.0, axis 0.0 0.0 1.0, limit lower=0.0 upper=1.5707963267948966 effort=50000 velocity=50000
- added joint l_hand_thumb_3_joint: type revolute, parent l_hand_thumb_2, child l_hand_thumb_3, origin xyz=0.022 0.0 0.0 rpy=0.0 0.0 0.0, axis 0.0 0.0 1.0, limit lower=0.0 upper=1.5707963267948966 effort=50000 velocity=50000
- joint l_hand_dh_frame_fixed_joint: axis (none) -> 0.0 0.0 1.0; limit (none) -> lower=0.0 upper=0.0 effort=50000 velocity=50000; type fixed -> revolute

Commit message: Implement right hand in iCubGazeboV2_5_vision_manip

File: iCub/robots/iCubGazeboV2_5_vision_manip/model.urdf (robot description, URDF)
Before this commit: robot iCub, 208 links, 207 joints
Links:
- added link r_hand_index_0, mass 0.01; collision mesh filename=package://iCub/meshes/hand/full_RightIndex0.obj scale=1.0 1.0 1.0; visual mesh filename=package://iCub/meshes/hand/full_RightIndex0.obj scale=1.0 1.0 1.0
- added link r_hand_index_1, mass 0.01; collision mesh filename=package://iCub/meshes/hand/full_RightIndex1.obj scale=1.0 1.0 1.0; visual mesh filename=package://iCub/meshes/hand/full_RightIndex1.obj scale=1.0 1.0 1.0
- added link r_hand_index_2, mass 0.01; collision mesh filename=package://iCub/meshes/hand/full_RightIndex2.obj scale=1.0 1.0 1.0; visual mesh filename=package://iCub/meshes/hand/full_RightIndex2.obj scale=1.0 1.0 1.0
- added link r_hand_index_3, mass 0.01; collision mesh filename=package://iCub/meshes/hand/full_RightIndex3.obj scale=1.0 1.0 1.0; visual mesh filename=package://iCub/meshes/hand/full_RightIndex3.obj scale=1.0 1.0 1.0
- added link r_hand_little_0, mass 0.01; collision mesh filename=package://iCub/meshes/hand/full_RightLittle0.obj scale=1.0 1.0 1.0; visual mesh filename=package://iCub/meshes/hand/full_RightLittle0.obj scale=1.0 1.0 1.0
- added link r_hand_little_1, mass 0.01; collision mesh filename=package://iCub/meshes/hand/full_RightLittle1.obj scale=1.0 1.0 1.0; visual mesh filename=package://iCub/meshes/hand/full_RightLittle1.obj scale=1.0 1.0 1.0
- added link r_hand_little_2, mass 0.01; collision mesh filename=package://iCub/meshes/hand/full_RightLittle2.obj scale=1.0 1.0 1.0; visual mesh filename=package://iCub/meshes/hand/full_RightLittle2.obj scale=1.0 1.0 1.0
- added link r_hand_little_3, mass 0.01; collision mesh filename=package://iCub/meshes/hand/full_RightLittle3.obj scale=1.0 1.0 1.0; visual mesh filename=package://iCub/meshes/hand/full_RightLittle3.obj scale=1.0 1.0 1.0
- added link r_hand_middle_0, mass 0.01; collision mesh filename=package://iCub/meshes/hand/full_RightMiddle0.obj scale=1.0 1.0 1.0; visual mesh filename=package://iCub/meshes/hand/full_RightMiddle0.obj scale=1.0 1.0 1.0
- added link r_hand_middle_1, mass 0.01; collision mesh filename=package://iCub/meshes/hand/full_RightMiddle1.obj scale=1.0 1.0 1.0; visual mesh filename=package://iCub/meshes/hand/full_RightMiddle1.obj scale=1.0 1.0 1.0
- added link r_hand_middle_2, mass 0.01; collision mesh filename=package://iCub/meshes/hand/full_RightMiddle2.obj scale=1.0 1.0 1.0; visual mesh filename=package://iCub/meshes/hand/full_RightMiddle2.obj scale=1.0 1.0 1.0
- added link r_hand_middle_3, mass 0.01; collision mesh filename=package://iCub/meshes/hand/full_RightMiddle3.obj scale=1.0 1.0 1.0; visual mesh filename=package://iCub/meshes/hand/full_RightMiddle3.obj scale=1.0 1.0 1.0
- added link r_hand_ring_0, mass 0.01; collision mesh filename=package://iCub/meshes/hand/full_RightRing0.obj scale=1.0 1.0 1.0; visual mesh filename=package://iCub/meshes/hand/full_RightRing0.obj scale=1.0 1.0 1.0
- added link r_hand_ring_1, mass 0.01; collision mesh filename=package://iCub/meshes/hand/full_RightRing1.obj scale=1.0 1.0 1.0; visual mesh filename=package://iCub/meshes/hand/full_RightRing1.obj scale=1.0 1.0 1.0
- added link r_hand_ring_2, mass 0.01; collision mesh filename=package://iCub/meshes/hand/full_RightRing2.obj scale=1.0 1.0 1.0; visual mesh filename=package://iCub/meshes/hand/full_RightRing2.obj scale=1.0 1.0 1.0
- added link r_hand_ring_3, mass 0.01; collision mesh filename=package://iCub/meshes/hand/full_RightRing3.obj scale=1.0 1.0 1.0; visual mesh filename=package://iCub/meshes/hand/full_RightRing3.obj scale=1.0 1.0 1.0
- added link r_hand_thumb_0, mass 0.01; collision mesh filename=package://iCub/meshes/hand/full_RightThumb0.obj scale=1.0 1.0 1.0; visual mesh filename=package://iCub/meshes/hand/full_RightThumb0.obj scale=1.0 1.0 1.0
- added link r_hand_thumb_1, mass 0.01; collision mesh filename=package://iCub/meshes/hand/full_RightThumb1.obj scale=1.0 1.0 1.0; visual mesh filename=package://iCub/meshes/hand/full_RightThumb1.obj scale=1.0 1.0 1.0
- added link r_hand_thumb_2, mass 0.01; collision mesh filename=package://iCub/meshes/hand/full_RightThumb2.obj scale=1.0 1.0 1.0; visual mesh filename=package://iCub/meshes/hand/full_RightThumb2.obj scale=1.0 1.0 1.0
- added link r_hand_thumb_3, mass 0.01; collision mesh filename=package://iCub/meshes/hand/full_RightThumb3.obj scale=1.0 1.0 1.0; visual mesh filename=package://iCub/meshes/hand/full_RightThumb3.obj scale=1.0 1.0 1.0
- link r_hand_dh_frame: mass None -> 0.001
Joints:
- added joint r_hand_index_0_joint: type revolute, parent r_hand_dh_frame, child r_hand_index_0, origin xyz=0.00175 -0.02622  -0.0107 rpy=3.05454839699628 -3.13536120039556 3.07030553260709, axis 0.0 0.0 -1.0, limit lower=0.0 upper=0.3490658503988659 effort=50000 velocity=50000
- added joint r_hand_index_1_joint: type revolute, parent r_hand_index_0, child r_hand_index_1, origin xyz=0.0148 0.00175 -1.07156594925393e-19 rpy=1.5707963267949 0.0 0.0, axis 0.0 0.0 1.0, limit lower=0.0 upper=1.5707963267948966 effort=50000 velocity=50000
- added joint r_hand_index_2_joint: type revolute, parent r_hand_index_1, child r_hand_index_2, origin xyz=0.0259 0.0 0.0 rpy=0.0 0.0 0.0, axis 0.0 0.0 1.0, limit lower=0.0 upper=1.5707963267948966 effort=50000 velocity=50000
- added joint r_hand_index_3_joint: type revolute, parent r_hand_index_2, child r_hand_index_3, origin xyz=0.022 0.0 0.0 rpy=0.0 0.0 0.0, axis 0.0 0.0 1.0, limit lower=0.0 upper=1.5707963267948966 effort=50000 velocity=50000
- added joint r_hand_little_0_joint: type revolute, parent r_hand_dh_frame, child r_hand_little_0, origin xyz=-0.000390000000000001 0.02454 -0.01 rpy=0.00929663374481331 0.0867711076126969 0.106868680136788, axis 0.0 0.0 1.0, limit lower=0.0 upper=0.3490658503988659 effort=50000 velocity=50000
- added joint r_hand_little_1_joint: type revolute, parent r_hand_little_0, child r_hand_little_1, origin xyz= 0.0148 -0.00175 1.07156594925393e-19 rpy=1.5707963267949 0.0 0.0, axis 0.0 0.0 1.0, limit lower=0.0 upper=1.5707963267948966 effort=50000 velocity=50000
- added joint r_hand_little_2_joint: type revolute, parent r_hand_little_1, child r_hand_little_2, origin xyz=0.0219 0.0 0.0 rpy=0.0 0.0 0.0, axis 0.0 0.0 1.0, limit lower=0.0 upper=1.5707963267948966 effort=50000 velocity=50000
- added joint r_hand_little_3_joint: type revolute, parent r_hand_little_2, child r_hand_little_3, origin xyz=0.019 0.0 0.0 rpy=0.0 0.0 0.0, axis 0.0 0.0 1.0, limit lower=0.0 upper=1.5707963267948966 effort=50000 velocity=50000
- added joint r_hand_middle_0_joint: type revolute, parent r_hand_dh_frame, child r_hand_middle_0, origin xyz=0.0025 -0.00977 -0.0116 rpy=0.0 0.0 0.0, axis 0.0 0.0 1.0, limit lower=0.0 upper=0.0 effort=50000 velocity=50000
- added joint r_hand_middle_1_joint: type revolute, parent r_hand_middle_0, child r_hand_middle_1, origin xyz=0.0153 0.0022 -1.34711147906209e-19 rpy=1.5707963267949 0.0 0.0, axis 0.0 0.0 1.0, limit lower=0.0 upper=1.5707963267948966 effort=50000 velocity=50000
- added joint r_hand_middle_2_joint: type revolute, parent r_hand_middle_1, child r_hand_middle_2, origin xyz=0.0258 0.0 0.0 rpy=0.0 0.0 0.0, axis 0.0 0.0 1.0, limit lower=0.0 upper=1.5707963267948966 effort=50000 velocity=50000
- added joint r_hand_middle_3_joint: type revolute, parent r_hand_middle_2, child r_hand_middle_3, origin xyz=0.024 0.0 0.0 rpy=0.0 0.0 0.0, axis 0.0 0.0 1.0, limit lower=0.0 upper=1.5707963267948966 effort=50000 velocity=50000
- added joint r_hand_ring_0_joint: type revolute, parent r_hand_dh_frame, child r_hand_ring_0, origin xyz=0.00163000000000001 0.00565 -0.011 rpy=0.00929663374481331 0.0867711076126969 0.106868680136788, axis 0.0 0.0 1.0, limit lower=0.0 upper=0.3490658503988659 effort=50000 velocity=50000
- added joint r_hand_ring_1_joint: type revolute, parent r_hand_ring_0, child r_hand_ring_1, origin xyz=0.0148 0.00175 -1.07156594925393e-19 rpy=1.5707963267949 0.0 0.0, axis 0.0 0.0 1.0, limit lower=0.0 upper=1.5707963267948966 effort=50000 velocity=50000
- added joint r_hand_ring_2_joint: type revolute, parent r_hand_ring_1, child r_hand_ring_2, origin xyz=0.0259 0.0 0.0 rpy=0.0 0.0 0.0, axis 0.0 0.0 1.0, limit lower=0.0 upper=1.5707963267948966 effort=50000 velocity=50000
- added joint r_hand_ring_3_joint: type revolute, parent r_hand_ring_2, child r_hand_ring_3, origin xyz=0.022 0.0 0.0 rpy=0.0 0.0 0.0, axis 0.0 0.0 1.0, limit lower=0.0 upper=1.5707963267948966 effort=50000 velocity=50000
- added joint r_hand_thumb_0_joint: type revolute, parent r_hand_dh_frame, child r_hand_thumb_0, origin xyz=-0.0235  -0.012 -0.0015 rpy=-1.6435245522555 3.10126979642577 2.07617279145347, axis 0.0 0.0 1.0, limit lower=0.0 upper=1.5707963267948966 effort=50000 velocity=50000
- added joint r_hand_thumb_1_joint: type revolute, parent r_hand_thumb_0, child r_hand_thumb_1, origin xyz=0.0211 0.0049 -3.00038465791102e-19 rpy=-1.5707963267949 0.0 0.0, axis 0.0 0.0 1.0, limit lower=0.0 upper=1.5707963267948966 effort=50000 velocity=50000
- added joint r_hand_thumb_2_joint: type revolute, parent r_hand_thumb_1, child r_hand_thumb_2, origin xyz=0.026 0.0 0.0 rpy=0.0 0.0 0.0, axis 0.0 0.0 1.0, limit lower=0.0 upper=1.5707963267948966 effort=50000 velocity=50000
- added joint r_hand_thumb_3_joint: type revolute, parent r_hand_thumb_2, child r_hand_thumb_3, origin xyz=0.022 0.0 0.0 rpy=0.0 0.0 0.0, axis 0.0 0.0 1.0, limit lower=0.0 upper=1.5707963267948966 effort=50000 velocity=50000
- joint r_hand_dh_frame_fixed_joint: axis (none) -> 0.0 0.0 1.0; limit (none) -> lower=0.0 upper=0.0 effort=50000 velocity=50000; type fixed -> revolute

Commit message: Fix robot to the root_link in iCubGazeboV2_5_vision_manip

File: iCub/robots/iCubGazeboV2_5_vision_manip/model.urdf (robot description, URDF)
Before this commit: robot iCub, 228 links, 227 joints
Links:
- added link world, mass 0.001
Joints:
- added joint world_to_root_link_joint: type revolute, parent world, child root_link, axis 0.0 0.0 1.0, limit lower=0.0 upper=0.0 effort=50000 velocity=50000
