Commit message: Clean iCubGazeboV2_5_vision_manip
Remove skin frames

Improve indentation

File: iCub/robots/iCubGazeboV2_5_vision_manip/model.urdf (robot description, URDF)
Before this commit: robot iCub, 229 links, 228 joints
Links:
- removed link imu_frame
- removed link l_forearm_skin_0
- removed link l_forearm_skin_1
- removed link l_forearm_skin_10
- removed link l_forearm_skin_11
- removed link l_forearm_skin_12
- removed link l_forearm_skin_13
- removed link l_forearm_skin_14
- removed link l_forearm_skin_15
- removed link l_forearm_skin_16
- removed link l_forearm_skin_17
- removed link l_forearm_skin_19
- removed link l_forearm_skin_2
- removed link l_forearm_skin_22
- removed link l_forearm_skin_24
- removed link l_forearm_skin_25
- removed link l_forearm_skin_28
- removed link l_forearm_skin_29
- removed link l_forearm_skin_3
- removed link l_forearm_skin_4
- removed link l_forearm_skin_5
- removed link l_forearm_skin_6
- removed link l_forearm_skin_7
- removed link l_forearm_skin_8
- removed link l_forearm_skin_9
- removed link l_sole
- removed link l_sole_skin_0
- removed link l_sole_skin_1
- removed link l_sole_skin_10
- removed link l_sole_skin_11
- removed link l_sole_skin_12
- removed link l_sole_skin_13
- removed link l_sole_skin_14
- removed link l_sole_skin_15
- removed link l_sole_skin_17
- removed link l_sole_skin_18
- removed link l_sole_skin_19
- removed link l_sole_skin_2
- removed link l_sole_skin_20
- removed link l_sole_skin_21
- removed link l_sole_skin_22
- removed link l_sole_skin_24
- removed link l_sole_skin_25
- removed link l_sole_skin_26
- removed link l_sole_skin_27
- removed link l_sole_skin_28
- removed link l_sole_skin_29
- removed link l_sole_skin_3
- removed link l_sole_skin_4
- removed link l_sole_skin_8
- removed link l_sole_skin_9
- removed link l_upper_leg_back_contact
- removed link r_forearm_skin_0
- removed link r_forearm_skin_1
- removed link r_forearm_skin_10
- removed link r_forearm_skin_11
- removed link r_forearm_skin_12
- removed link r_forearm_skin_13
- removed link r_forearm_skin_14
- removed link r_forearm_skin_15
- removed link r_forearm_skin_16
- removed link r_forearm_skin_17
- removed link r_forearm_skin_19
- removed link r_forearm_skin_2
- removed link r_forearm_skin_22
- removed link r_forearm_skin_24
- removed link r_forearm_skin_25
- removed link r_forearm_skin_28
- removed link r_forearm_skin_29
- removed link r_forearm_skin_3
- removed link r_forearm_skin_4
- removed link r_forearm_skin_5
- removed link r_forearm_skin_6
- removed link r_forearm_skin_7
- removed link r_forearm_skin_8
- removed link r_forearm_skin_9
- removed link r_lower_leg_skin_0
- removed link r_lower_leg_skin_10
- removed link r_lower_leg_skin_11
- removed link r_lower_leg_skin_14
- removed link r_lower_leg_skin_15
- removed link r_lower_leg_skin_16
- removed link r_lower_leg_skin_17
- removed link r_lower_leg_skin_19
- removed link r_lower_leg_skin_20
- removed link r_lower_leg_skin_21
- removed link r_lower_leg_skin_28
- removed link r_lower_leg_skin_29
- removed link r_lower_leg_skin_3
- removed link r_lower_leg_skin_31
- removed link r_lower_leg_skin_32
- removed link r_lower_leg_skin_35
- removed link r_lower_leg_skin_36
- removed link r_lower_leg_skin_37
- removed link r_lower_leg_skin_38
- removed link r_lower_leg_skin_4
- removed link r_lower_leg_skin_41
- removed link r_lower_leg_skin_42
- removed link r_lower_leg_skin_43
- removed link r_lower_leg_skin_46
- removed link r_lower_leg_skin_47
- removed link r_lower_leg_skin_49
- removed link r_lower_leg_skin_5
- removed link r_lower_leg_skin_50
- removed link r_lower_leg_skin_51
- removed link r_lower_leg_skin_52
- removed link r_lower_leg_skin_53
- removed link r_lower_leg_skin_54
- removed link r_lower_leg_skin_55
- removed link r_lower_leg_skin_56
- removed link r_lower_leg_skin_6
- removed link r_lower_leg_skin_60
- removed link r_lower_leg_skin_61
- removed link r_lower_leg_skin_9
- removed link r_sole
- removed link r_sole_skin_0
- removed link r_sole_skin_1
- removed link r_sole_skin_10
- removed link r_sole_skin_11
- removed link r_sole_skin_12
- removed link r_sole_skin_13
- removed link r_sole_skin_14
- removed link r_sole_skin_15
- removed link r_sole_skin_17
- removed link r_sole_skin_18
- removed link r_sole_skin_19
- removed link r_sole_skin_2
- removed link r_sole_skin_20
- removed link r_sole_skin_21
- removed link r_sole_skin_22
- removed link r_sole_skin_24
- removed link r_sole_skin_25
- removed link r_sole_skin_26
- removed link r_sole_skin_27
- removed link r_sole_skin_28
- removed link r_sole_skin_29
- removed link r_sole_skin_3
- removed link r_sole_skin_4
- removed link r_sole_skin_8
- removed link r_sole_skin_9
- removed link r_upper_leg_back_contact
Joints:
- removed joint imu_frame_fixed_joint
- removed joint l_forearm_skin_0_fixed_joint
- removed joint l_forearm_skin_10_fixed_joint
- removed joint l_forearm_skin_11_fixed_joint
- removed joint l_forearm_skin_12_fixed_joint
- removed joint l_forearm_skin_13_fixed_joint
- removed joint l_forearm_skin_14_fixed_joint
- removed joint l_forearm_skin_15_fixed_joint
- removed joint l_forearm_skin_16_fixed_joint
- removed joint l_forearm_skin_17_fixed_joint
- removed joint l_forearm_skin_19_fixed_joint
- removed joint l_forearm_skin_1_fixed_joint
- removed joint l_forearm_skin_22_fixed_joint
- removed joint l_forearm_skin_24_fixed_joint
- removed joint l_forearm_skin_25_fixed_joint
- removed joint l_forearm_skin_28_fixed_joint
- removed joint l_forearm_skin_29_fixed_joint
- removed joint l_forearm_skin_2_fixed_joint
- removed joint l_forearm_skin_3_fixed_joint
- removed joint l_forearm_skin_4_fixed_joint
- removed joint l_forearm_skin_5_fixed_joint
- removed joint l_forearm_skin_6_fixed_joint
- removed joint l_forearm_skin_7_fixed_joint
- removed joint l_forearm_skin_8_fixed_joint
- removed joint l_forearm_skin_9_fixed_joint
- removed joint l_sole_fixed_joint
- removed joint l_sole_skin_0_fixed_joint
- removed joint l_sole_skin_10_fixed_joint
- removed joint l_sole_skin_11_fixed_joint
- removed joint l_sole_skin_12_fixed_joint
- removed joint l_sole_skin_13_fixed_joint
- removed joint l_sole_skin_14_fixed_joint
- removed joint l_sole_skin_15_fixed_joint
- removed joint l_sole_skin_17_fixed_joint
- removed joint l_sole_skin_18_fixed_joint
- removed joint l_sole_skin_19_fixed_joint
- removed joint l_sole_skin_1_fixed_joint
- removed joint l_sole_skin_20_fixed_joint
- removed joint l_sole_skin_21_fixed_joint
- removed joint l_sole_skin_22_fixed_joint
- removed joint l_sole_skin_24_fixed_joint
- removed joint l_sole_skin_25_fixed_joint
- removed joint l_sole_skin_26_fixed_joint
- removed joint l_sole_skin_27_fixed_joint
- removed joint l_sole_skin_28_fixed_joint
- removed joint l_sole_skin_29_fixed_joint
- removed joint l_sole_skin_2_fixed_joint
- removed joint l_sole_skin_3_fixed_joint
- removed joint l_sole_skin_4_fixed_joint
- removed joint l_sole_skin_8_fixed_joint
- removed joint l_sole_skin_9_fixed_joint
- removed joint l_upper_leg_back_contact_fixed_joint
- removed joint r_forearm_skin_0_fixed_joint
- removed joint r_forearm_skin_10_fixed_joint
- removed joint r_forearm_skin_11_fixed_joint
- removed joint r_forearm_skin_12_fixed_joint
- removed joint r_forearm_skin_13_fixed_joint
- removed joint r_forearm_skin_14_fixed_joint
- removed joint r_forearm_skin_15_fixed_joint
- removed joint r_forearm_skin_16_fixed_joint
- removed joint r_forearm_skin_17_fixed_joint
- removed joint r_forearm_skin_19_fixed_joint
- removed joint r_forearm_skin_1_fixed_joint
- removed joint r_forearm_skin_22_fixed_joint
- removed joint r_forearm_skin_24_fixed_joint
- removed joint r_forearm_skin_25_fixed_joint
- removed joint r_forearm_skin_28_fixed_joint
- removed joint r_forearm_skin_29_fixed_joint
- removed joint r_forearm_skin_2_fixed_joint
- removed joint r_forearm_skin_3_fixed_joint
- removed joint r_forearm_skin_4_fixed_joint
- removed joint r_forearm_skin_5_fixed_joint
- removed joint r_forearm_skin_6_fixed_joint
- removed joint r_forearm_skin_7_fixed_joint
- removed joint r_forearm_skin_8_fixed_joint
- removed joint r_forearm_skin_9_fixed_joint
- removed joint r_lower_leg_skin_0_fixed_joint
- removed joint r_lower_leg_skin_10_fixed_joint
- removed joint r_lower_leg_skin_11_fixed_joint
- removed joint r_lower_leg_skin_14_fixed_joint
- removed joint r_lower_leg_skin_15_fixed_joint
- removed joint r_lower_leg_skin_16_fixed_joint
- removed joint r_lower_leg_skin_17_fixed_joint
- removed joint r_lower_leg_skin_19_fixed_joint
- removed joint r_lower_leg_skin_20_fixed_joint
- removed joint r_lower_leg_skin_21_fixed_joint
- removed joint r_lower_leg_skin_28_fixed_joint
- removed joint r_lower_leg_skin_29_fixed_joint
- removed joint r_lower_leg_skin_31_fixed_joint
- removed joint r_lower_leg_skin_32_fixed_joint
- removed joint r_lower_leg_skin_35_fixed_joint
- removed joint r_lower_leg_skin_36_fixed_joint
- removed joint r_lower_leg_skin_37_fixed_joint
- removed joint r_lower_leg_skin_38_fixed_joint
- removed joint r_lower_leg_skin_3_fixed_joint
- removed joint r_lower_leg_skin_41_fixed_joint
- removed joint r_lower_leg_skin_42_fixed_joint
- removed joint r_lower_leg_skin_43_fixed_joint
- removed joint r_lower_leg_skin_46_fixed_joint
- removed joint r_lower_leg_skin_47_fixed_joint
- removed joint r_lower_leg_skin_49_fixed_joint
- removed joint r_lower_leg_skin_4_fixed_joint
- removed joint r_lower_leg_skin_50_fixed_joint
- removed joint r_lower_leg_skin_51_fixed_joint
- removed joint r_lower_leg_skin_52_fixed_joint
- removed joint r_lower_leg_skin_53_fixed_joint
- removed joint r_lower_leg_skin_54_fixed_joint
- removed joint r_lower_leg_skin_55_fixed_joint
- removed joint r_lower_leg_skin_56_fixed_joint
- removed joint r_lower_leg_skin_5_fixed_joint
- removed joint r_lower_leg_skin_60_fixed_joint
- removed joint r_lower_leg_skin_61_fixed_joint
- removed joint r_lower_leg_skin_6_fixed_joint
- removed joint r_lower_leg_skin_9_fixed_joint
- removed joint r_sole_fixed_joint
- removed joint r_sole_skin_0_fixed_joint
- removed joint r_sole_skin_10_fixed_joint
- removed joint r_sole_skin_11_fixed_joint
- removed joint r_sole_skin_12_fixed_joint
- removed joint r_sole_skin_13_fixed_joint
- removed joint r_sole_skin_14_fixed_joint
- removed joint r_sole_skin_15_fixed_joint
- removed joint r_sole_skin_17_fixed_joint
- removed joint r_sole_skin_18_fixed_joint
- removed joint r_sole_skin_19_fixed_joint
- removed joint r_sole_skin_1_fixed_joint
- removed joint r_sole_skin_20_fixed_joint
- removed joint r_sole_skin_21_fixed_joint
- removed joint r_sole_skin_22_fixed_joint
- removed joint r_sole_skin_24_fixed_joint
- removed joint r_sole_skin_25_fixed_joint
- removed joint r_sole_skin_26_fixed_joint
- removed joint r_sole_skin_27_fixed_joint
- removed joint r_sole_skin_28_fixed_joint
- removed joint r_sole_skin_29_fixed_joint
- removed joint r_sole_skin_2_fixed_joint
- removed joint r_sole_skin_3_fixed_joint
- removed joint r_sole_skin_4_fixed_joint
- removed joint r_sole_skin_8_fixed_joint
- removed joint r_sole_skin_9_fixed_joint
- removed joint r_upper_leg_back_contact_fixed_joint

Commit message: Add fake inertias to DH kinematic frames in iCubGazeboV2_5_vision_manip

File: iCub/robots/iCubGazeboV2_5_vision_manip/model.urdf (robot description, URDF)
Before this commit: robot iCub, 88 links, 87 joints
Links:
- link l_foot_dh_frame: mass None -> 0.001
- link l_forearm_dh_frame: mass None -> 0.001
- link l_upper_leg_dh_frame: mass None -> 0.001
- link r_foot_dh_frame: mass None -> 0.001
- link r_forearm_dh_frame: mass None -> 0.001
- link r_upper_leg_dh_frame: mass None -> 0.001

Commit message: Add kinematic frames for finger tips
Fake inertias have been added to these frames

The value 0.0168 is from icub iKinFwd

File: iCub/robots/iCubGazeboV2_5_vision_manip/model.urdf (robot description, URDF)
Before this commit: robot iCub, 88 links, 87 joints
Links:
- added link l_hand_index_tip, mass 0.001
- added link l_hand_little_tip, mass 0.001
- added link l_hand_middle_tip, mass 0.001
- added link l_hand_ring_tip, mass 0.001
- added link l_hand_thumb_tip, mass 0.001
- added link r_hand_index_tip, mass 0.001
- added link r_hand_little_tip, mass 0.001
- added link r_hand_middle_tip, mass 0.001
- added link r_hand_ring_tip, mass 0.001
- added link r_hand_thumb_tip, mass 0.001
Joints:
- added joint l_hand_index_tip_joint: type revolute, parent l_hand_index_3, child l_hand_index_tip, origin xyz=0.0168 0.0 0.0 rpy=-1.5707963267948966 0.0 0.0, axis 0.0 0.0 1.0, limit lower=0.0 upper=0.0 effort=50000 velocity=50000
- added joint l_hand_little_tip_joint: type revolute, parent l_hand_little_3, child l_hand_little_tip, origin xyz=0.0168 0.0 0.0 rpy=-1.5707963267948966 0.0 0.0, axis 0.0 0.0 1.0, limit lower=0.0 upper=0.0 effort=50000 velocity=50000
- added joint l_hand_middle_tip_joint: type revolute, parent l_hand_middle_3, child l_hand_middle_tip, origin xyz=0.0168 0.0 0.0 rpy=-1.5707963267948966 0.0 0.0, axis 0.0 0.0 1.0, limit lower=0.0 upper=0.0 effort=50000 velocity=50000
- added joint l_hand_ring_tip_joint: type revolute, parent l_hand_ring_3, child l_hand_ring_tip, origin xyz=0.0168 0.0 0.0 rpy=-1.5707963267948966 0.0 0.0, axis 0.0 0.0 1.0, limit lower=0.0 upper=0.0 effort=50000 velocity=50000
- added joint l_hand_thumb_tip_joint: type revolute, parent l_hand_thumb_3, child l_hand_thumb_tip, origin xyz=0.0168 0.0 0.0 rpy=-1.5707963267948966 0.0 0.0, axis 0.0 0.0 1.0, limit lower=0.0 upper=0.0 effort=50000 velocity=50000
- added joint r_hand_index_tip_joint: type revolute, parent r_hand_index_3, child r_hand_index_tip, origin xyz=0.0168 0.0 0.0 rpy=-1.5707963267948966 0.0 0.0, axis 0.0 0.0 1.0, limit lower=0.0 upper=0.0 effort=50000 velocity=50000
- added joint r_hand_little_tip_joint: type revolute, parent r_hand_little_3, child r_hand_little_tip, origin xyz=0.0168 0.0 0.0 rpy=-1.5707963267948966 0.0 0.0, axis 0.0 0.0 1.0, limit lower=0.0 upper=0.0 effort=50000 velocity=50000
- added joint r_hand_middle_tip_joint: type revolute, parent r_hand_middle_3, child r_hand_middle_tip, origin xyz=0.0168 0.0 0.0 rpy=-1.5707963267948966 0.0 0.0, axis 0.0 0.0 1.0, limit lower=0.0 upper=0.0 effort=50000 velocity=50000
- added joint r_hand_ring_tip_joint: type revolute, parent r_hand_ring_3, child r_hand_ring_tip, origin xyz=0.0168 0.0 0.0 rpy=-1.5707963267948966 0.0 0.0, axis 0.0 0.0 1.0, limit lower=0.0 upper=0.0 effort=50000 velocity=50000
- added joint r_hand_thumb_tip_joint: type revolute, parent r_hand_thumb_3, child r_hand_thumb_tip, origin xyz=0.0168 0.0 0.0 rpy=-1.5707963267948966 0.0 0.0, axis 0.0 0.0 1.0, limit lower=0.0 upper=0.0 effort=50000 velocity=50000

Commit message: Fix axis direction for joints l_hand_{ring, little}_0_joint in iCubGazeboV2_5_vision_manip

File: iCub/robots/iCubGazeboV2_5_vision_manip/model.urdf (robot description, URDF)
Before this commit: robot iCub, 98 links, 97 joints
Joints:
- joint l_hand_little_0_joint: axis 0.0 0.0 1.0 -> 0.0 0.0 -1.0
- joint l_hand_ring_0_joint: axis 0.0 0.0 1.0 -> 0.0 0.0 -1.0
