Commit message: Use simplified meshes for collision of fingers in iCubGazeboV2_5_vision_manip

File: iCub/robots/iCubGazeboV2_5_vision_manip/model.urdf (robot description, URDF)
Before this commit: robot iCub, 98 links, 97 joints
Links:
- link l_hand: geometry collision mesh filename=package://iCub/meshes/hand/col_LeftHandPalm.obj scale=1.0 1.0 1.0; visual mesh filename=package://iCub/meshes/hand/full_LeftHandPalm.obj scale=1.0 1.0 1.0
- link l_hand_index_0: geometry collision mesh filename=package://iCub/meshes/hand/col_LeftIndex0.obj scale=1.0 1.0 1.0; visual mesh filename=package://iCub/meshes/hand/full_LeftIndex0.obj scale=1.0 1.0 1.0
- link l_hand_index_1: geometry collision mesh filename=package://iCub/meshes/hand/col_LeftIndex1.obj scale=1.0 1.0 1.0; visual mesh filename=package://iCub/meshes/hand/full_LeftIndex1.obj scale=1.0 1.0 1.0
- link l_hand_index_2: geometry collision mesh filename=package://iCub/meshes/hand/col_LeftIndex2.obj scale=1.0 1.0 1.0; visual mesh filename=package://iCub/meshes/hand/full_LeftIndex2.obj scale=1.0 1.0 1.0
- link l_hand_index_3: geometry collision mesh filename=package://iCub/meshes/hand/col_LeftIndex3.obj scale=1.0 1.0 1.0; visual mesh filename=package://iCub/meshes/hand/full_LeftIndex3.obj scale=1.0 1.0 1.0
- link l_hand_little_0: geometry collision mesh filename=package://iCub/meshes/hand/col_LeftLittle0.obj scale=1.0 1.0 1.0; visual mesh filename=package://iCub/meshes/hand/full_LeftLittle0.obj scale=1.0 1.0 1.0
- link l_hand_little_1: geometry collision mesh filename=package://iCub/meshes/hand/full_LeftLittle1.obj scale=1.0 1.0 1.0; visual mesh filename=package://iCub/meshes/hand/col_LeftLittle1.obj scale=1.0 1.0 1.0
- link l_hand_little_2: geometry collision mesh filename=package://iCub/meshes/hand/col_LeftLittle2.obj scale=1.0 1.0 1.0; visual mesh filename=package://iCub/meshes/hand/full_LeftLittle2.obj scale=1.0 1.0 1.0
- link l_hand_little_3: geometry collision mesh filename=package://iCub/meshes/hand/col_LeftLittle3.obj scale=1.0 1.0 1.0; visual mesh filename=package://iCub/meshes/hand/full_LeftLittle3.obj scale=1.0 1.0 1.0
- link l_hand_middle_0: geometry collision mesh filename=package://iCub/meshes/hand/col_LeftMiddle0.obj scale=1.0 1.0 1.0; visual mesh filename=package://iCub/meshes/hand/full_LeftMiddle0.obj scale=1.0 1.0 1.0
- link l_hand_middle_1: geometry collision mesh filename=package://iCub/meshes/hand/col_LeftMiddle1.obj scale=1.0 1.0 1.0; visual mesh filename=package://iCub/meshes/hand/full_LeftMiddle1.obj scale=1.0 1.0 1.0
- link l_hand_middle_2: geometry collision mesh filename=package://iCub/meshes/hand/col_LeftMiddle2.obj scale=1.0 1.0 1.0; visual mesh filename=package://iCub/meshes/hand/full_LeftMiddle2.obj scale=1.0 1.0 1.0
- link l_hand_middle_3: geometry collision mesh filename=package://iCub/meshes/hand/col_LeftMiddle3.obj scale=1.0 1.0 1.0; visual mesh filename=package://iCub/meshes/hand/full_LeftMiddle3.obj scale=1.0 1.0 1.0
- link l_hand_ring_0: geometry collision mesh filename=package://iCub/meshes/hand/col_LeftRing0.obj scale=1.0 1.0 1.0; visual mesh filename=package://iCub/meshes/hand/full_LeftRing0.obj scale=1.0 1.0 1.0
- link l_hand_ring_1: geometry collision mesh filename=package://iCub/meshes/hand/col_LeftRing1.obj scale=1.0 1.0 1.0; visual mesh filename=package://iCub/meshes/hand/full_LeftRing1.obj scale=1.0 1.0 1.0
- link l_hand_ring_2: geometry collision mesh filename=package://iCub/meshes/hand/col_LeftRing2.obj scale=1.0 1.0 1.0; visual mesh filename=package://iCub/meshes/hand/full_LeftRing2.obj scale=1.0 1.0 1.0
- link l_hand_ring_3: geometry collision mesh filename=package://iCub/meshes/hand/col_LeftRing3.obj scale=1.0 1.0 1.0; visual mesh filename=package://iCub/meshes/hand/full_LeftRing3.obj scale=1.0 1.0 1.0
- link l_hand_thumb_0: geometry collision mesh filename=package://iCub/meshes/hand/col_LeftThumb0.obj scale=1.0 1.0 1.0; visual mesh filename=package://iCub/meshes/hand/full_LeftThumb0.obj scale=1.0 1.0 1.0
- link l_hand_thumb_1: geometry collision mesh filename=package://iCub/meshes/hand/col_LeftThumb1.obj scale=1.0 1.0 1.0; visual mesh filename=package://iCub/meshes/hand/full_LeftThumb1.obj scale=1.0 1.0 1.0
- link l_hand_thumb_2: geometry collision mesh filename=package://iCub/meshes/hand/col_LeftThumb2.obj scale=1.0 1.0 1.0; visual mesh filename=package://iCub/meshes/hand/col_LeftThumb2.obj scale=1.0 1.0 1.0
- link l_hand_thumb_3: geometry collision mesh filename=package://iCub/meshes/hand/col_LeftThumb3.obj scale=1.0 1.0 1.0; visual mesh filename=package://iCub/meshes/hand/full_LeftThumb3.obj scale=1.0 1.0 1.0
- link r_hand: geometry collision mesh filename=package://iCub/meshes/hand/col_RightHandPalm.obj scale=1.0 1.0 1.0; visual mesh filename=package://iCub/meshes/hand/full_RightHandPalm.obj scale=1.0 1.0 1.0
- link r_hand_index_0: geometry collision mesh filename=package://iCub/meshes/hand/col_RightIndex0.obj scale=1.0 1.0 1.0; visual mesh filename=package://iCub/meshes/hand/full_RightIndex0.obj scale=1.0 1.0 1.0
- link r_hand_index_1: geometry collision mesh filename=package://iCub/meshes/hand/col_RightIndex1.obj scale=1.0 1.0 1.0; visual mesh filename=package://iCub/meshes/hand/full_RightIndex1.obj scale=1.0 1.0 1.0
- link r_hand_index_2: geometry collision mesh filename=package://iCub/meshes/hand/col_RightIndex2.obj scale=1.0 1.0 1.0; visual mesh filename=package://iCub/meshes/hand/full_RightIndex2.obj scale=1.0 1.0 1.0
- link r_hand_index_3: geometry collision mesh filename=package://iCub/meshes/hand/col_RightIndex3.obj scale=1.0 1.0 1.0; visual mesh filename=package://iCub/meshes/hand/full_RightIndex3.obj scale=1.0 1.0 1.0
- link r_hand_little_0: geometry collision mesh filename=package://iCub/meshes/hand/col_RightLittle0.obj scale=1.0 1.0 1.0; visual mesh filename=package://iCub/meshes/hand/full_RightLittle0.obj scale=1.0 1.0 1.0
- link r_hand_little_1: geometry collision mesh filename=package://iCub/meshes/hand/col_RightLittle1.obj scale=1.0 1.0 1.0; visual mesh filename=package://iCub/meshes/hand/full_RightLittle1.obj scale=1.0 1.0 1.0
- link r_hand_little_2: geometry collision mesh filename=package://iCub/meshes/hand/col_RightLittle2.obj scale=1.0 1.0 1.0; visual mesh filename=package://iCub/meshes/hand/full_RightLittle2.obj scale=1.0 1.0 1.0
- link r_hand_little_3: geometry collision mesh filename=package://iCub/meshes/hand/col_RightLittle3.obj scale=1.0 1.0 1.0; visual mesh filename=package://iCub/meshes/hand/full_RightLittle3.obj scale=1.0 1.0 1.0
- link r_hand_middle_0: geometry collision mesh filename=package://iCub/meshes/hand/col_RightMiddle0.obj scale=1.0 1.0 1.0; visual mesh filename=package://iCub/meshes/hand/full_RightMiddle0.obj scale=1.0 1.0 1.0
- link r_hand_middle_1: geometry collision mesh filename=package://iCub/meshes/hand/col_RightMiddle1.obj scale=1.0 1.0 1.0; visual mesh filename=package://iCub/meshes/hand/full_RightMiddle1.obj scale=1.0 1.0 1.0
- link r_hand_middle_2: geometry collision mesh filename=package://iCub/meshes/hand/col_RightMiddle2.obj scale=1.0 1.0 1.0; visual mesh filename=package://iCub/meshes/hand/full_RightMiddle2.obj scale=1.0 1.0 1.0
- link r_hand_middle_3: geometry collision mesh filename=package://iCub/meshes/hand/col_RightMiddle3.obj scale=1.0 1.0 1.0; visual mesh filename=package://iCub/meshes/hand/full_RightMiddle3.obj scale=1.0 1.0 1.0
- link r_hand_ring_0: geometry collision mesh filename=package://iCub/meshes/hand/col_RightRing0.obj scale=1.0 1.0 1.0; visual mesh filename=package://iCub/meshes/hand/full_RightRing0.obj scale=1.0 1.0 1.0
- link r_hand_ring_1: geometry collision mesh filename=package://iCub/meshes/hand/col_RightRing1.obj scale=1.0 1.0 1.0; visual mesh filename=package://iCub/meshes/hand/full_RightRing1.obj scale=1.0 1.0 1.0
- link r_hand_ring_2: geometry collision mesh filename=package://iCub/meshes/hand/col_RightRing2.obj scale=1.0 1.0 1.0; visual mesh filename=package://iCub/meshes/hand/full_RightRing2.obj scale=1.0 1.0 1.0
- link r_hand_ring_3: geometry collision mesh filename=package://iCub/meshes/hand/col_RightRing3.obj scale=1.0 1.0 1.0; visual mesh filename=package://iCub/meshes/hand/full_RightRing3.obj scale=1.0 1.0 1.0
- link r_hand_thumb_0: geometry collision mesh filename=package://iCub/meshes/hand/col_RightThumb0.obj scale=1.0 1.0 1.0; visual mesh filename=package://iCub/meshes/hand/full_RightThumb0.obj scale=1.0 1.0 1.0
- link r_hand_thumb_1: geometry collision mesh filename=package://iCub/meshes/hand/col_RightThumb1.obj scale=1.0 1.0 1.0; visual mesh filename=package://iCub/meshes/hand/full_RightThumb1.obj scale=1.0 1.0 1.0
- link r_hand_thumb_2: geometry collision mesh filename=package://iCub/meshes/hand/col_RightThumb2.obj scale=1.0 1.0 1.0; visual mesh filename=package://iCub/meshes/hand/full_RightThumb2.obj scale=1.0 1.0 1.0
- link r_hand_thumb_3: geometry collision mesh filename=package://iCub/meshes/hand/col_RightThumb3.obj scale=1.0 1.0 1.0; visual mesh filename=package://iCub/meshes/hand/full_RightThumb3.obj scale=1.0 1.0 1.0

Commit message: Implement eyes in iCubGazeboV2_5_vision_manip

File: iCub/robots/iCubGazeboV2_5_vision_manip/model.urdf (robot description, URDF)
Before this commit: robot iCub, 98 links, 97 joints
Links:
- added link eyes_tilt_frame, mass 0.001
- added link l_eye, mass 0.01; visual cylinder length=0.001 radius=0.008; visual sphere radius=0.02
- added link r_eye, mass 0.01; visual cylinder length=0.001 radius=0.008; visual sphere radius=0.02
Joints:
- added joint eyes_tilt: type revolute, parent head, child eyes_tilt_frame, origin xyz=1.90392435799427e-10 0.104896999999692 0.0455907000018309 rpy=-2.35618706953753 1.57079632678797 0.785405584052268, axis 0.0 0.0 1.0, limit lower=-0.5235987755982988 upper=0.5235987755982988 effort=50000 velocity=50000
- added joint l_eye_pan_joint: type revolute, parent eyes_tilt_frame, child l_eye, origin xyz=0.0 0.0 -0.034 rpy=0.0 -1.5707963267949 0.0, axis 0.0 1.0 0.0, limit lower=-0.5235987755982988 upper=0.9599310885968813 effort=50000 velocity=50000
- added joint r_eye_pan_joint: type revolute, parent eyes_tilt_frame, child r_eye, origin xyz=0.0 0.0 0.034 rpy=0.0 -1.5707963267949 0.0, axis 0.0 1.0 0.0, limit lower=-0.9599310885968813 upper=0.5235987755982988 effort=50000 velocity=50000

Commit message: Finalize visual configuration of eye bulbs

File: iCub/robots/iCubGazeboV2_5_vision_manip/model.urdf (robot description, URDF)
Before this commit: robot iCub, 101 links, 100 joints
Links:
- link l_eye: geometry visual cylinder length=0.001 radius=0.005; visual sphere radius=0.02
- link r_eye: geometry visual cylinder length=0.001 radius=0.005; visual sphere radius=0.02

Commit message: Fix wrong axis direction for joint r_wrist_yaw

File: iCub/robots/iCubGazeboV2_5_vision_manip/model.urdf (robot description, URDF)
Before this commit: robot iCub, 101 links, 100 joints
Joints:
- joint r_wrist_yaw: axis 2.22044604925e-16 1.0 0.0 -> 2.22044604925e-16 -1.0 0.0
